File: DRV10987_SAMD21uC_V1.5/DRV10987.sch (EAGLE design)
At the start: 75 parts, among them J1 SUCHAI_PCB, J10 455-1750-1-ND, J7 MK1_ZERO_ZX62AB-5PA(11), U1 MK1_ZERO_AP7215-33YG-13, U2 ATSAMD21G-A, Y1 32.768kHz

Commit message: new SAMD21uC_v1.5, added BTS5045, molex connectors, remove conf jumpers, and added holes for wires
Parts:
- removed J10: 455-1750-1-ND, SparkFun-Connectors:CONN_03
- removed J12, J15, J16, J17: (no value), SparkFun-Connectors:CONN_01
- removed J13, J18, J4, J5, J6: (no value), SparkFun-Connectors:CONN_03LOCK
- removed J2: (no value), SparkFun-Connectors:CONN_05LOCK_LONGPADS
- removed R4: 1k, resistors-longpads:1KOHM-HORIZ-1/4W-5%
- removed R5: 2k, resistors-longpads:RESISTORAXIAL-0.3
- removed U$4: WIRELESS-BLUETOOTH-HC-05-MIRRORMIRROR, diy-modules:WIRELESS-BLUETOOTH-HC-05-MIRRORMIRROR
- added J8: (no value), SparkFun-Connectors:CONN_03LOCK
- added U3: BTS5045-1EJA, BTS5045-1EJA:BTS5045-1EJA
- added X1, X3, X4: 53398-03, con-molex:53398-03
- added X2: 53398-05, con-molex:53398-05
Connections:
- removed net 11.1V_LIPO: J10.3, J13.3
- removed net I2C2_SCL: J1.6, J19.3
- removed net I2C2_SDA: J1.5, J18.3
- removed net I2C_SCL: J1.22, J19.1
- removed net I2C_SDA: J1.21, J18.1
- removed net MCU-RX: U$4.TX
- removed net MCU-TX: R4.2
- removed net N$13: R4.1, R5.2, U$4.RX
- new net BTS_VS: J14.2, J8.2, U3.VS
- new net N$12: U$2.IN+, U3.OUT1, U3.OUT2, U3.OUT3
- new net RWS_DEN: J1.15, U3.DEN
- new net RWS_EN: J1.16, U3.IN
- new net RWS_IS: J1.14, U3.IS
- net +5V: no longer U$4.+5V
- net 12V_REG: now also S2.P; no longer J13.1
- net 3V3: now also X2-2.S; no longer J2.2
- net 5V_OUT_STACK: now also J11.1, J14.3, J8.3; no longer J12.1, J15.1
- net 5V_STACK: no longer J14.3
- net GND: now also J19.1, U3.GND, X2-3.S; no longer J10.1, J2.3, R5.1, U$4.GND
- net I2C_SCL_UC: now also J1.5, J19.3; no longer J19.2
- net I2C_SDA_UC: now also J1.6, J19.2; no longer J18.2
- net N$16: now also J1.21; no longer J13.2, J16.1, S2.P
- net N$18: now also J1.22; no longer J14.2, U$2.IN+
- net N$5: no longer J17.1
- net OUT1: now also X1-1.S; no longer J4.1
- net OUT1_M2: now also X3-1.S; no longer J5.1
- net OUT1_M3: now also X4-1.S; no longer J6.1
- net OUT2: now also X1-2.S; no longer J4.2
- net OUT2_M2: now also X3-2.S; no longer J5.2
- net OUT2_M3: now also X4-2.S; no longer J6.2
- net OUT3: now also X1-3.S; no longer J4.3
- net OUT3_M2: now also X3-3.S; no longer J5.3
- net OUT3_M3: now also X4-3.S; no longer J6.3
- net RESET: now also X2-1.S; no longer J2.1
- net SWCLK: now also X2-4.S; no longer J2.4
- net SWDIO: now also X2-5.S; no longer J2.5
- net V_BATT_STACK: now also J8.1
Other:
- moved on the sheet: C10, C11, C12, C13, C14, C16, C17, C18, C7, C8, C9, J11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

Commit message: added rtc, atmega328, leds, labels and adjust usb connector
Parts:
- added C32, C33: 22pF, SparkFun-Capacitors:22PF-0603-50V-5%
- added C34: 1nF, SparkFun-Capacitors:1.0NF/1000PF-0603-50V-10%
- added C35, C36: 1.0uF, SparkFun-Capacitors:1.0UF-0402-16V-10%
- added D1: RED, SparkFun-LED:LED-RED0603
- added D2, D4, D5: BLUE, SparkFun-LED:LED-BLUE0603
- added D3: GREEN, SparkFun-LED:LED-GREEN0603
- added Q2: (no value), adafruit:XTAL-4-3225
- added R14, R8: (no value), adafruit:R-US_R0402
- added R15, R17, R19, R20: 22, SparkFun-Resistors:22OHM-0603-1/10W-1%
- added R16, R4: 100K, SparkFun-Resistors:100KOHM-0402-1/16W-1%
- added R18: 1k, SparkFun-Resistors:1KOHM-0603-1/10W-1%
- added R5: 10k, SparkFun-Resistors:10KOHM-0603-1/10W-1%
- added RTC1: DS3231M, SparkFun-Clocks:DS3231M
- added U$4: (no value), adafruit:CR1220SMT
- added U4: ATMEGA328P_TQFP, SparkFun-IC-Microcontroller:ATMEGA328P_TQFP
- added X6: 53398-06, con-molex:53398-06
- added X7: 53398-05, con-molex:53398-05
Connections:
- new net AT328-RX: U4.PD0(RXD), X7-1.S
- new net AT328-TX: U4.PD1(TXD), X7-2.S
- new net AT328_MISO: U4.PB4(MISO), X6-2.S
- new net AT328_MOSI: U4.PB3(MOSI/OC2), X6-1.S
- new net AT328_RESET: R5.1, U4.PC6(/RESET), X6-5.S, X7-4.S
- new net AT328_SCK: U4.PB5(SCK), X6-3.S
- new net N$13: C32.2, Q2.X1, U4.PB6(XTAL1/TOSC1)
- new net N$14: C33.2, Q2.X2, U4.PB7(XTAL2/TOSC2)
- new net N$15: D1.A, R15.1
- new net N$21: D2.A, R17.2
- new net N$36: D3.A, R18.1
- new net N$37: D4.A, R19.2
- new net N$38: R19.1, U2.PA15(XOUT/SER2:3+)
- new net N$39: D5.A, R20.2
- new net N$40: R20.1, U4.PD5(T1)
- new net RTC_32KHZ: R4.1, RTC1.32KHZ, U4.PD3(INT1)
- new net RTC_BAT: C34.1, C36.1, RTC1.VBAT, U$4.+, U$4.+1
- new net RTC_INT: R16.1, RTC1.SQW, U4.PD2(INT0)
- new net RTC_RST: RTC1.RST, U4.ADC6
- new net RTC_SCL: R8.1, RTC1.SCL, U4.PC5(ADC5/SCL)
- new net RTC_SDA: R14.1, RTC1.SDA, U4.PC4(ADC4/SDA)
- net +5V: now also C35.1, R14.2, R16.2, R17.1, R4.2, R5.2, R8.2, RTC1.VCC, U4.AVCC, U4.VCC@4, U4.VCC@6, X6-4.S, X7-3.S
- net 12V: now also R18.2
- net 3V3: now also R15.2
- net GND: now also C32.1, C33.1, C34.2, C35.2, C36.2, D1.C, D2.C, D3.C, D4.C, D5.C, Q2.G1, Q2.G2, RTC1.GND, U$4.-, U4.GND@3, U4.GND@5, X6-6.S, X7-5.S
- net RWS_DEN: now also U4.PC0(ADC0); no longer J1.15
- net RWS_EN: now also U4.PC1(ADC1); no longer J1.16
- net RWS_IS: now also U4.ADC7; no longer J1.14
Other:
- moved on the sheet: C10, C11, C12, C13, C16, C17, C18, C9, J11, J14, J3, J7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
